File: hardware/usb-hub.kicad_pcb (KiCad board)
At the start: 4 copper layers, 61.4 x 45.8 mm, 72 parts, among them J1 USB_C_Receptacle, J2 USB_C_Receptacle, J3 USB_C_Receptacle, J4 USB_C_Receptacle, J5 USB_C_Receptacle, U1 TUSB8041, U2 TPS2561, U3 TPS2561, U4 HD3S3220, U5 HD3S3220, U6 MCP1700x-330xxTT, U7 HD3S3220, U8 HD3S3220, U9 HD3S3220, Y1 Crystal_GND24

Commit message: pcb updated
Parts:
- removed the G*** at (119.9, 70.7)
- added G***: LOGO, LOGO, F.Cu at (99.6, 86.2)
- added G***: LOGO, LOGO, B.Cu at (127.7, 87.8)
- added G***: LOGO, LOGO, B.Cu at (114.7, 66.0)
- added REF**: LayerMarker_4_6.35x2.54mm_TextH1mm_P1.27mm, Symbol:LayerMarker_4_6.35x2.54mm_TextH1mm_P1.27mm, F.Cu at (133.9, 54.2)
- moved G*** 23.3 mm to (114.8, 83.7)
- moved G*** 1.41 mm to (94.6, 57.6)
Other:
- board text added: "5 gigabits per second btw"
- board text added: "bits go brrrr"
- board text added: "if you can read this, you have voided your warranty"
