File: hardware/usb-hub.kicad_sch (KiCad schematic)
At the start: 1 part, among them U1 TUSB8041

Commit message: Hello World
Parts:
- added C1, C10, C11, C2, C3, C4, C5, C6, C7, C8, C9: 100n, Capacitor_SMD:C_0402_1005Metric, symbol Device:C_Small
- added C12, C13: C_Small, Capacitor_SMD:C_0402_1005Metric, symbol Device:C_Small
- added J1, J2, J3, J4, J5: USB_C_Receptacle, Connector_USB:USB_C_Receptacle_Molex_105450-0101, symbol Connector:USB_C_Receptacle
- added R1: 9.53k, Resistor_SMD:R_0402_1005Metric, symbol Device:R_Small
- added R10, R11, R12, R13, R14, R15, R16, R17, R18, R19: 5.1k, Resistor_SMD:R_0402_1005Metric, symbol Device:R_Small
- added R2, R3, R4: 4.7k, Resistor_SMD:R_0402_1005Metric, symbol Device:R_Small
- added R5: 10k, Resistor_SMD:R_0402_1005Metric, symbol Device:R_Small
- added R6: 90.9k, Resistor_SMD:R_0402_1005Metric, symbol Device:R_Small
- added R7: 1M, Resistor_SMD:R_0402_1005Metric, symbol Device:R
- added R8, R9: 30k, Resistor_SMD:R_0402_1005Metric, symbol Device:R_Small
- added U2, U3: TPS2561, Package_SON:VSON-10-1EP_3x3mm_P0.5mm_EP1.65x2.4mm_ThermalVias, symbol Interface_USB:TPS2561
- added Y1: Crystal_GND24, Crystal:Crystal_SMD_3225-4Pin_3.2x2.5mm, symbol Device:Crystal_GND24
Connections:
- net USB1_DP: now reaches U1.1 (USB_DP_DN1)
- net USB1_DP: now also J2.A6 (D+), J2.B6 (D+)
- net USB2_DN: now reaches U1.10 (USB_DM_DN2)
- net USB2_DN: now also J3.A7 (D-), J3.B7 (D-)
- net TX_2P: now reaches U1.11 (USB_SSTXP_DN2)
- net TX_2P: now also C3.1
- net TX_2N: now reaches U1.12 (USB_SSTXM_DN2)
- net TX_2N: now also C4.1
- net +1V1: now reaches U1.13 (VDD)
- net +1V1: now also U1.21 (VDD), U1.28 (VDD), U1.31 (VDD), U1.5 (VDD), U1.51 (VDD), U1.57 (VDD), U1.8 (VDD)
- net SSRX2P: now reaches U1.14 (USB_SSRXP_DN2)
- net SSRX2P: now also J3.B11 (RX1+)
- net SSRX2N: now reaches U1.15 (USB_SSRXM_DN2)
- net SSRX2N: now also J3.B10 (RX1-)
- net +3V3: now reaches U1.16 (VDD33)
- net +3V3: now also U1.34 (VDD33), U1.52 (VDD33), U1.63 (VDD33)
- net USB3_DP: now reaches U1.17 (USB_DP_DN3)
- net USB3_DP: now also J4.A6 (D+), J4.B6 (D+)
- net USB3_DN: now reaches U1.18 (USB_DM_DN3)
- net USB3_DN: now also J4.A7 (D-), J4.B7 (D-)
- net TX_3P: now reaches U1.19 (USB_SSTXP_DN3)
- net TX_3P: now also C5.1
- net USB1_DN: now reaches U1.2 (USB_DM_DN1)
- net USB1_DN: now also J2.A7 (D-), J2.B7 (D-)
- net TX_3N: now reaches U1.20 (USB_SSTXM_DN3)
- net TX_3N: now also C6.1
- net SSRX3P: now reaches U1.22 (USB_SSRXP_DN3)
- net SSRX3P: now also J4.B11 (RX1+)
- net SSRX3N: now reaches U1.23 (USB_SSRXM_DN3)
- net SSRX3N: now also J4.B10 (RX1-)
- net USB4_DP: now reaches U1.24 (USB_DP_DN4)
- net USB4_DP: now also J5.A6 (D+), J5.B6 (D+)
- net USB4_DN: now reaches U1.25 (USB_DM_DN4)
- net USB4_DN: now also J5.A7 (D-), J5.B7 (D-)
- net TX_4P: now reaches U1.26 (USB_SSTXP_DN4)
- net TX_4P: now also C7.1
- net TX_4N: now reaches U1.27 (USB_SSTXM_DN4)
- net TX_4N: now also C8.1
- net SSRX4P: now reaches U1.29 (USB_SSRXP_DN4)
- net SSRX4P: now also J5.B11 (RX1+)
- net TX_1P: now reaches U1.3 (USB_SSTXP_DN1)
- net TX_1P: now also C1.1
- net SSRX4N: now reaches U1.30 (USB_SSRXM_DN4)
- net SSRX4N: now also J5.B10 (RX1-)
- net CTRL_4: now reaches U1.32 (PWRCTL4/BATEN4)
- net CTRL_4: now also U3.5 (EN2)
- net CTRL_3: now reaches U1.33 (PWRCTL3/BATEN3)
- net CTRL_3: now also U3.4 (EN1)
- net CTRL_2: now reaches U1.35 (PWRCTL2/BATEN2)
- net CTRL_2: now also U2.5 (EN2)
- net CTRL_1: now reaches U1.36 (PWRCTL1/BATEN1)
- net CTRL_1: now also U2.4 (EN1)
- net TX_1N: now reaches U1.4 (USB_SSTXM_DN1)
- net TX_1N: now also C2.1
- net at U1.42 (GANGED/SMBA2/HS_UP): now also R4.1
- net at U1.45 (AUTOENz/HS_SUSPEND): now also R3.1
- net at U1.48 (USB_VBUS): now also R5.1, R6.2
- net at U1.49 (TEST): now also R2.1
- net at U1.50 (GRSTz): now also C11.2
- net USBUP_DN: now reaches U1.53 (USB_DP_UP)
- net USBUP_DN: now also J1.A7 (D-), J1.B7 (D-)
- net USBUP_DP: now reaches U1.54 (USB_DM_UP)
- net USBUP_DP: now also J1.A6 (D+), J1.B6 (D+)
- net TX_0P: now reaches U1.55 (USB_SSTXP_UP)
- net TX_0P: now also C9.2
- net TX_0N: now reaches U1.56 (USB_SSTXM_UP)
- net TX_0N: now also C10.2
- net SSRXUPP: now reaches U1.58 (USB_SSRXP_UP)
- net SSRXUPP: now also J1.B11 (RX1+)
- net SSRXUPN: now reaches U1.59 (USB_SSRXM_UP)
- net SSRXUPN: now also J1.B10 (RX1-)
- net SSRX1P: now reaches U1.6 (USB_SSRXP_DN1)
- net SSRX1P: now also J2.B11 (RX1+)
- net XO: now reaches U1.61 (XO)
- net XO: now also C12.1, R7.1, Y1.1
- net XI: now reaches U1.62 (XI)
- net XI: now also C13.1, R7.2, Y1.3
- net at U1.64 (USB_R1): now also R1.1
- net GND: now reaches U1.65 (VSS)
- net GND: now also C11.1, C12.2, C13.2, J1.A1 (GND), J1.A12 (GND), J1.B1 (GND), J1.B12 (GND), J1.SH (SHIELD), J2.A1 (GND), J2.A12 (GND), J2.B1 (GND), J2.B12 (GND), J2.SH (SHIELD), J3.A1 (GND), J3.A12 (GND), J3.B1 (GND), J3.B12 (GND), J3.SH (SHIELD), J4.A1 (GND), J4.A12 (GND), J4.B1 (GND), J4.B12 (GND), J4.SH (SHIELD), J5.A1 (GND), J5.A12 (GND), J5.B1 (GND), J5.B12 (GND), J5.SH (SHIELD), R1.2, R10.2, R11.2, R2.2, R3.2, R4.2, R5.2, R8.2, R9.2, U2.1 (GND), U2.11 (PAD), U3.1 (GND), U3.11 (PAD), Y1.2 (G), Y1.4 (G)
- net SSRX1N: now reaches U1.7 (USB_SSRXM_DN1)
- net SSRX1N: now also J2.B10 (RX1-)
- net USB2_DP: now reaches U1.9 (USB_DP_DN2)
- net USB2_DP: now also J3.A6 (D+), J3.B6 (D+)
- new net: J5.A5 (CC1), R19.2
- new net: J5.B5 (CC2), R18.2
- new net: R8.1, U2.7 (ILM)
- new net: J4.B5 (CC2), R16.2
- new net: J2.A5 (CC1), R13.2
- new net: J2.B5 (CC2), R12.2
- new net: J4.A5 (CC1), R17.2
- new net: J3.A5 (CC1), R15.2
- new net: J1.A5 (CC1), R11.1
- new net: J1.B5 (CC2), R10.1
- new net: R9.1, U3.7 (ILM)
- new net: J3.B5 (CC2), R14.2
- new net SSTX1N: C2.2, J2.A3 (TX1-)
- new net SSTX1P: C1.2, J2.A2 (TX1+)
- new net SSTX2N: C4.2, J3.A3 (TX1-)
- new net SSTX2P: C3.2, J3.A2 (TX1+)
- new net SSTX3N: C6.2, J4.A3 (TX1-)
- new net SSTX3P: C5.2, J4.A2 (TX1+)
- new net SSTX4N: C8.2, J5.A3 (TX1-)
- new net SSTX4P: C7.2, J5.A2 (TX1+)
- new net SSTXUPN: C10.1, J1.A3 (TX1-)
- new net SSTXUPP: C9.1, J1.A2 (TX1+)
- new net VBUS: J1.A4 (VBUS), J1.A9 (VBUS), J1.B4 (VBUS), J1.B9 (VBUS), R6.1, U2.2 (IN), U2.3 (IN), U3.2 (IN), U3.3 (IN)
- new net VBUS_1: J2.A4 (VBUS), J2.A9 (VBUS), J2.B4 (VBUS), J2.B9 (VBUS), R12.1, R13.1, U2.9 (OUT1)
- new net VBUS_2: J3.A4 (VBUS), J3.A9 (VBUS), J3.B4 (VBUS), J3.B9 (VBUS), R14.1, R15.1, U2.8 (OUT2)
- new net VBUS_3: J4.A4 (VBUS), J4.A9 (VBUS), J4.B4 (VBUS), J4.B9 (VBUS), R16.1, R17.1, U3.9 (OUT1)
- new net VBUS_4: J5.A4 (VBUS), J5.A9 (VBUS), J5.B4 (VBUS), J5.B9 (VBUS), R18.1, R19.1, U3.8 (OUT2)
- no-connect marks 0 -> 43
Other:
- note added: "+-1%"
- moved on the sheet: U1

Commit message: PCB Changed
Parts:
- removed C10, C5, C6, C7, C8, C9: 100n, Capacitor_SMD:C_0402_1005Metric, symbol Device:C_Small
- removed R14, R15, R16, R17, R18, R19: 5.1k, Resistor_SMD:R_0402_1005Metric, symbol Device:R_Small
- added C14, C15, C16, C17, C18, C19, C20, C21, C22, C23, C24, C25, C26, C27, C28, C29: 100n, Capacitor_SMD:C_0402_1005Metric, symbol Device:C_Small
- added C5, C8: 10u, Capacitor_SMD:C_0603_1608Metric, symbol Device:C
- added C6, C7: 100n, Capacitor_SMD:C_0402_1005Metric, symbol Device:C
- added H1, H2, H3, H4: MountingHole, MountingHole:MountingHole_2.2mm_M2, symbol Mechanical:MountingHole
- added R20, R21, R25, R27, R29: 100k, Resistor_SMD:R_0402_1005Metric, symbol Device:R_Small
- added R22, R23, R24, R26, R28: 900k, Resistor_SMD:R_0402_1005Metric, symbol Device:R_Small
- added U4, U5, U7, U8, U9: HD3S3220, Package_DFN_QFN:Texas_RNH0030A_WQFN-30-1EP_2.5x4.5mm_P0.4mm_EP1.2x3.2mm, symbol Interface_USB:HD3S3220
- added U6: MCP1700x-330xxTT, Package_TO_SOT_SMD:SOT-23, symbol Regulator_Linear:MCP1700x-330xxTT
- R10, R11, R12, R13: value 5.1k -> 10k
Connections:
- net TX_3N is gone; now on net SSTX3N: U1.20 (USB_SSTXM_DN3)
- net TX_3P is gone; now on net SSTX3P: U1.19 (USB_SSTXP_DN3)
- net TX_4N is gone; now on net SSTX4N: U1.27 (USB_SSTXM_DN4)
- net TX_4P is gone; now on net SSTX4P: U1.26 (USB_SSTXP_DN4)
- net +3V3: now also C7.1, C8.1, R20.1, R21.1, R25.1, R27.1, R29.1, U4.8 (VCC33), U5.8 (VCC33), U6.2 (VO), U7.8 (VCC33), U8.8 (VCC33), U9.8 (VCC33)
- net GND: now also C5.2, C6.2, C7.2, C8.2, U4.12 (ENn_MUX), U4.13 (GND), U4.28 (GND), U4.29 (ENn_CC), U4.31 (EP), U4.4 (PORT), U5.12 (ENn_MUX), U5.13 (GND), U5.28 (GND), U5.29 (ENn_CC), U5.31 (EP), U6.1 (GND), U7.12 (ENn_MUX), U7.13 (GND), U7.28 (GND), U7.29 (ENn_CC), U7.31 (EP), U8.12 (ENn_MUX), U8.13 (GND), U8.28 (GND), U8.29 (ENn_CC), U8.31 (EP), U9.12 (ENn_MUX), U9.13 (GND), U9.28 (GND), U9.29 (ENn_CC), U9.31 (EP); no longer R10.2, R11.2
- net SSRX1N: now also U5.9 (RXP); no longer J2.B10 (RX1-)
- net SSRX1P: now also U5.10 (RXN); no longer J2.B11 (RX1+)
- net SSRX2N: now also U7.9 (RXP); no longer J3.B10 (RX1-)
- net SSRX2P: now also U7.10 (RXN); no longer J3.B11 (RX1+)
- net SSRX3N: now also U8.9 (RXP); no longer J4.B10 (RX1-)
- net SSRX3P: now also U8.10 (RXN); no longer J4.B11 (RX1+)
- net SSRX4N: now also U9.9 (RXP); no longer J5.B10 (RX1-)
- net SSRX4P: now also U9.10 (RXN); no longer J5.B11 (RX1+)
- net SSTX1N: now also U1.4 (USB_SSTXM_DN1), U5.6 (TXP); no longer C2.2, J2.A3 (TX1-)
- net SSTX1P: now also U1.3 (USB_SSTXP_DN1), U5.7 (TXN); no longer C1.2, J2.A2 (TX1+)
- net SSTX2N: now also U1.12 (USB_SSTXM_DN2), U7.6 (TXP); no longer C4.2, J3.A3 (TX1-)
- net SSTX2P: now also U1.11 (USB_SSTXP_DN2), U7.7 (TXN); no longer C3.2, J3.A2 (TX1+)
- net SSTX3N: now also U8.6 (TXP); no longer J4.A3 (TX1-)
- net SSTX3P: now also U8.7 (TXN); no longer J4.A2 (TX1+)
- net SSTX4N: now also U9.6 (TXP); no longer J5.A3 (TX1-)
- net SSTX4P: now also U9.7 (TXN); no longer J5.A2 (TX1+)
- net VBUS: now also C5.1, C6.1, R22.1, U4.30 (VDD5), U6.3 (VI)
- net VBUS_1: now also R10.1, R23.1, U5.30 (VDD5), U5.4 (PORT); no longer R12.1, R13.1
- net VBUS_2: now also R11.1, R24.1, U7.30 (VDD5), U7.4 (PORT)
- net VBUS_3: now also R12.1, R26.1, U8.30 (VDD5), U8.4 (PORT)
- net VBUS_4: now also R13.1, R28.1, U9.30 (VDD5), U9.4 (PORT)
- net DFP4RX2N: now reaches J5.A10 (RX2-)
- net DFP4RX2N: now also U9.18 (RX2N)
- net DFP4RX2P: now reaches J5.A11 (RX2+)
- net DFP4RX2P: now also U9.19 (RX2P)
- net at J5.A5 (CC1): now also U9.2 (CC1)
- net 4TX2P: now reaches J5.B2 (TX2+)
- net 4TX2P: now also C24.2
- net 4TX2N: now reaches J5.B3 (TX2-)
- net 4TX2N: now also C22.2
- net at J5.B5 (CC2): now also U9.1 (CC2)
- net at J4.B5 (CC2): now also U8.1 (CC2)
- net DFP1RX2N: now reaches J2.A10 (RX2-)
- net DFP1RX2N: now also U5.18 (RX2N)
- net DFP1RX2P: now reaches J2.A11 (RX2+)
- net DFP1RX2P: now also U5.19 (RX2P)
- net at R13.2: now also U9.3 (CURRENT_MODE); no longer J2.A5 (CC1)
- net 1TX2P: now reaches J2.B2 (TX2+)
- net 1TX2P: now also C3.2
- net 1TX2N: now reaches J2.B3 (TX2-)
- net 1TX2N: now also C4.2
- net at J2.B5 (CC2): now also U5.1 (CC2); no longer R12.2
- net at J4.A5 (CC1): now also U8.2 (CC1)
- net at J3.A5 (CC1): now also U7.2 (CC1)
- net at J1.A5 (CC1): now also U4.2 (CC1); no longer R11.1
- net at J1.B5 (CC2): now also U4.1 (CC2); no longer R10.1
- net UFPRX2N: now reaches J1.A10 (RX2-)
- net UFPRX2N: now also U4.18 (RX2N)
- net UFPRX2P: now reaches J1.A11 (RX2+)
- net UFPRX2P: now also U4.19 (RX2P)
- net 0UFPTX2P: now reaches J1.B2 (TX2+)
- net 0UFPTX2P: now also C29.2
- net 0UFPTX2N: now reaches J1.B3 (TX2-)
- net 0UFPTX2N: now also C28.2
- net DFP3RX2N: now reaches J4.A10 (RX2-)
- net DFP3RX2N: now also U8.18 (RX2N)
- net DFP3RX2P: now reaches J4.A11 (RX2+)
- net DFP3RX2P: now also U8.19 (RX2P)
- net 3TX2P: now reaches J4.B2 (TX2+)
- net 3TX2P: now also C20.2
- net 3TX2N: now reaches J4.B3 (TX2-)
- net 3TX2N: now also C18.2
- net DFP2RX2N: now reaches J3.A10 (RX2-)
- net DFP2RX2N: now also U7.18 (RX2N)
- net DFP2RX2P: now reaches J3.A11 (RX2+)
- net DFP2RX2P: now also U7.19 (RX2P)
- net 2TX2P: now reaches J3.B2 (TX2+)
- net 2TX2P: now also C16.2
- net 2TX2N: now reaches J3.B3 (TX2-)
- net 2TX2N: now also C14.2
- net at J3.B5 (CC2): now also U7.1 (CC2)
- net SSRXUPN renamed SSRXUFPN
- net SSRXUFPN: now also U4.9 (RXP); no longer J1.B10 (RX1-)
- net SSRXUPP renamed SSRXUFPP
- net SSRXUFPP: now also U4.10 (RXN); no longer J1.B11 (RX1+)
- net SSTXUPN renamed 0UFPTX1P
- net 0UFPTX1P: now also C27.2
- net SSTXUPP renamed 0UFPTX1N
- net 0UFPTX1N: now also C26.2
- net TX_0N renamed SSTXUFPN
- net SSTXUFPN: now also U4.6 (TXP)
- net TX_0P renamed SSTXUFPP
- net SSTXUFPP: now also U4.7 (TXN)
- net TX_1N renamed DFP1TX1P
- net DFP1TX1P: now also U5.17 (TX1P); no longer U1.4 (USB_SSTXM_DN1)
- net TX_1P renamed DFP1TX1N
- net DFP1TX1N: now also U5.16 (TX1N); no longer U1.3 (USB_SSTXP_DN1)
- net TX_2N renamed DFP1TX2P
- net DFP1TX2P: now also U5.21 (TX2P); no longer U1.12 (USB_SSTXM_DN2)
- net TX_2P renamed DFP1TX2N
- net DFP1TX2N: now also U5.20 (TX2N); no longer U1.11 (USB_SSTXP_DN2)
- net USBUP_DN renamed USBUFP_DN
- net USBUP_DP renamed USBUFP_DP
- new net: R26.2, U8.5 (VBUS_DET)
- new net: R29.2, U9.11 (DIR)
- new net: R24.2, U7.5 (VBUS_DET)
- new net: R25.2, U7.11 (DIR)
- new net: J2.A5 (CC1), U5.2 (CC1)
- new net: R11.2, U7.3 (CURRENT_MODE)
- new net: R20.2, U5.11 (DIR)
- new net: R10.2, U5.3 (CURRENT_MODE)
- new net: R23.2, U5.5 (VBUS_DET)
- new net: R22.2, U4.5 (VBUS_DET)
- new net: R21.2, U4.11 (DIR)
- new net: R27.2, U8.11 (DIR)
- new net: R28.2, U9.5 (VBUS_DET)
- new net: R12.2, U8.3 (CURRENT_MODE)
- new net 1TX1N: C1.2, J2.A2 (TX1+)
- new net 1TX1P: C2.2, J2.A3 (TX1-)
- new net 2TX1N: C15.2, J3.A2 (TX1+)
- new net 2TX1P: C17.2, J3.A3 (TX1-)
- new net 3TX1N: C19.2, J4.A2 (TX1+)
- new net 3TX1P: C21.2, J4.A3 (TX1-)
- new net 4TX1N: C23.2, J5.A2 (TX1+)
- new net 4TX1P: C25.2, J5.A3 (TX1-)
- new net DFP1RX1N: J2.B10 (RX1-), U5.14 (RX1N)
- new net DFP1RX1P: J2.B11 (RX1+), U5.15 (RX1P)
- new net DFP2RX1N: J3.B10 (RX1-), U7.14 (RX1N)
- new net DFP2RX1P: J3.B11 (RX1+), U7.15 (RX1P)
- new net DFP2TX1N: C15.1, U7.16 (TX1N)
- new net DFP2TX1P: C17.1, U7.17 (TX1P)
- new net DFP2TX2N: C14.1, U7.20 (TX2N)
- new net DFP2TX2P: C16.1, U7.21 (TX2P)
- new net DFP3RX1N: J4.B10 (RX1-), U8.14 (RX1N)
- new net DFP3RX1P: J4.B11 (RX1+), U8.15 (RX1P)
- new net DFP3TX1N: C19.1, U8.16 (TX1N)
- new net DFP3TX1P: C21.1, U8.17 (TX1P)
- new net DFP3TX2N: C18.1, U8.20 (TX2N)
- new net DFP3TX2P: C20.1, U8.21 (TX2P)
- new net DFP4RX1N: J5.B10 (RX1-), U9.14 (RX1N)
- new net DFP4RX1P: J5.B11 (RX1+), U9.15 (RX1P)
- new net DFP4TX1N: C23.1, U9.16 (TX1N)
- new net DFP4TX1P: C25.1, U9.17 (TX1P)
- new net DFP4TX2N: C22.1, U9.20 (TX2N)
- new net DFP4TX2P: C24.1, U9.21 (TX2P)
- new net UFPRX1N: J1.B10 (RX1-), U4.14 (RX1N)
- new net UFPRX1P: J1.B11 (RX1+), U4.15 (RX1P)
- new net UFPTX1N: C26.1, U4.16 (TX1N)
- new net UFPTX1P: C27.1, U4.17 (TX1P)
- new net UFPTX2N: C28.1, U4.20 (TX2N)
- new net UFPTX2P: C29.1, U4.21 (TX2P)
- no-connect marks 43 -> 54
Other:
- moved on the sheet: J2
